File: KiCad/NR23_Schematic_v1.0/Microcontroller.kicad_sch (KiCad schematic)
At the start: 0 parts

Commit message: microcontroller
Parts:
- added U?: TI_J12_CANbus, symbol Homssymbols:TI_J12_CANbus
- added U?: TI_J1/J3, symbol Homssymbols:TI_J1/J3
Changed lines of the file:
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@@
 (kicad_sch (version 20211123) (generator eeschema)
   (paper "A")
+  (symbol (lib_id "Homssymbols:TI_J12_CANbus") (at 109.22 158.75 0) (unit 1)
+    (in_bom yes) (on_board yes) (fields_autoplaced)
+    (property "Reference" "U?" (id 0) (at 125.73 150.4949 0)
+      (effects (font (size 1.27 1.27)) (justify left))
+    )
+    (property "Value" "TI_J12_CANbus" (id 1) (at 125.73 153.0349 0)
+      (effects (font (size 1.27 1.27)) (justify left))
+    )
+    (property "Footprint" "" (id 2) (at 109.22 158.75 0)
+      (effects (font (size 1.27 1.27)) hide)
+    )
+    (property "Datasheet" "" (id 3) (at 109.22 158.75 0)
+      (effects (font (size 1.27 1.27)) hide)
+    )
+    (pin "")
+    (pin "")
+    (pin "J12")
+  )
+  (symbol (lib_id "Homssymbols:TI_J1{slash}J3") (at 106.68 115.57 0) (unit 1)
+    (in_bom yes) (on_board yes) (fields_autoplaced)
+    (property "Reference" "U?" (id 0) (at 95.25 74.93 0))
+    (property "Value" "TI_J1/J3" (id 1) (at 95.25 77.47 0))
+    (property "Footprint" "" (id 2) (at 125.73 120.65 0)
+      (effects (font (size 1.27 1.27)) hide)
+    )
+    (property "Datasheet" "" (id 3) (at 125.73 120.65 0)
+      (effects (font (size 1.27 1.27)) hide)
+    )
+    (pin "J1/01")
+    (pin "J1/03")
+    (pin "J1/04")
+    (pin "J3/21")
+    (pin "J3/22")
+  )
 )

Commit message: microcontroller
Parts:
- added U?: CANbus, symbol Homssymbols:CANbus
Other:
- moved on the sheet: U?
Changed lines of the file:
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@@
 (kicad_sch (version 20211123) (generator eeschema)
   (paper "A")
-  (symbol (lib_id "Homssymbols:TI_J12_CANbus") (at 109.22 158.75 0) (unit 1)
+  (symbol (lib_id "Homssymbols:CANbus") (at 135.89 151.13 0) (unit 1)
     (in_bom yes) (on_board yes) (fields_autoplaced)
-    (property "Reference" "U?" (id 0) (at 125.73 150.4949 0)
+    (property "Reference" "U?" (id 0) (at 167.64 149.8599 0)
       (effects (font (size 1.27 1.27)) (justify left))
     )
-    (property "Value" "TI_J12_CANbus" (id 1) (at 125.73 153.0349 0)
+    (property "Value" "CANbus" (id 1) (at 167.64 152.3999 0)
       (effects (font (size 1.27 1.27)) (justify left))
     )
-    (property "Footprint" "" (id 2) (at 109.22 158.75 0)
+    (property "Footprint" "" (id 2) (at 142.24 146.05 0)
       (effects (font (size 1.27 1.27)) hide)
     )
-    (property "Datasheet" "" (id 3) (at 109.22 158.75 0)
+    (property "Datasheet" "" (id 3) (at 142.24 146.05 0)
       (effects (font (size 1.27 1.27)) hide)
     )
+    (pin "")
+    (pin "")
+    (pin "")
+  )
+  (symbol (lib_id "Homssymbols:TI_J12_CANbus") (at 125.73 127 0) (unit 1)
+    (in_bom yes) (on_board yes) (fields_autoplaced)
+    (property "Reference" "U?" (id 0) (at 142.24 118.7449 0)
+      (effects (font (size 1.27 1.27)) (justify left))
+    )
+    (property "Value" "TI_J12_CANbus" (id 1) (at 142.24 121.2849 0)
+      (effects (font (size 1.27 1.27)) (justify left))
+    )
+    (property "Footprint" "" (id 2) (at 125.73 127 0)
+      (effects (font (size 1.27 1.27)) hide)
+    )
+    (property "Datasheet" "" (id 3) (at 125.73 127 0)
+      (effects (font (size 1.27 1.27)) hide)
+    )

Commit message: microcontroller + symbol library
Parts:
- removed U?: CANbus, symbol Homssymbols:CANbus
- added U?: TI_Board, symbol Homssymbols:TI_Board
- added U?: CANbus, symbol Homssymbols:CANbus
Connections:
- net GND: now reaches U?. (GND)
- net GND: now also U?. (To_TI_CAN_L)
- new net: U?. (GND), U?. (To_TI_CAN_L) (x2)
Changed lines of the file:
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@@
 (kicad_sch (version 20211123) (generator eeschema)
   (paper "A")
-  (symbol (lib_id "Homssymbols:CANbus") (at 135.89 151.13 0) (unit 1)
-    (in_bom yes) (on_board yes) (fields_autoplaced)
-    (property "Reference" "U?" (id 0) (at 167.64 149.8599 0)
-      (effects (font (size 1.27 1.27)) (justify left))
-    )
-    (property "Value" "CANbus" (id 1) (at 167.64 152.3999 0)
-      (effects (font (size 1.27 1.27)) (justify left))
-    )
-    (property "Footprint" "" (id 2) (at 142.24 146.05 0)
-      (effects (font (size 1.27 1.27)) hide)
-    )
-    (property "Datasheet" "" (id 3) (at 142.24 146.05 0)
-      (effects (font (size 1.27 1.27)) hide)
-    )
-    (pin "")
-    (pin "")
-    (pin "")
+  (wire (pts (xy 137.16 140.97) (xy 137.16 125.73))
+    (stroke (width 0) (type default) (color 0 0 0 0))
+  )
+  (wire (pts (xy 102.87 138.43) (xy 134.62 138.43))
+    (stroke (width 0) (type default) (color 0 0 0 0))
+  )
+  (wire (pts (xy 134.62 138.43) (xy 134.62 125.73))
+    (stroke (width 0) (type default) (color 0 0 0 0))
+  )
+  (wire (pts (xy 102.87 140.97) (xy 137.16 140.97))
+    (stroke (width 0) (type default) (color 0 0 0 0))
   )
   (symbol (lib_id "Homssymbols:TI_J12_CANbus") (at 125.73 127 0) (unit 1)
@@
     (pin "")
     (pin "")
-    (pin "J12")
+    (pin "")
+  )
+  (symbol (lib_id "Homssymbols:TI_Board") (at 134.62 87.63 0) (unit 1)
+    (in_bom yes) (on_board yes) (fields_autoplaced)
+    (property "Reference" "U?" (id 0) (at 210.82 90.1699 0)
+      (effects (font (size 1.27 1.27)) (justify left))
+    )
+    (property "Value" "TI_Board" (id 1) (at 210.82 92.7099 0)
+      (effects (font (size 1.27 1.27)) (justify left))
+    )
+    (property "Footprint" "" (id 2) (at 134.62 87.63 0)
+      (effects (font (size 1.27 1.27)) hide)
+    )
+    (property "Datasheet" "" (id 3) (at 134.62 87.63 0)
+      (effects (font (size 1.27 1.27)) hide)
+    )
+  )
+  (symbol (lib_id "power:GND") (at 77.47 163.83 0) (unit 1)
+    (in_bom yes) (on_board yes) (fields_autoplaced)
+    (property "Reference" "#PWR?" (id 0) (at 77.47 170.18 0)
+      (effects (font (size 1.27 1.27)) hide)
+    )
+    (property "Value" "GND" (id 1) (at 77.47 168.91 0))
+    (property "Footprint" "" (id 2) (at 77.47 163.83 0)
+      (effects (font (size 1.27 1.27)) hide)
+    )
+    (property "Datasheet" "" (id 3) (at 77.47 163.83 0)
+      (effects (font (size 1.27 1.27)) hide)
+    )
+    (pin "1")
+  )
+  (symbol (lib_id "power:GND") (at 132.08 125.73 0) (unit 1)
+    (in_bom yes) (on_board yes) (fields_autoplaced)
+    (property "Reference" "#PWR?" (id 0) (at 132.08 132.08 0)
+      (effects (font (size 1.27 1.27)) hide)
+    )
+    (property "Value" "GND" (id 1) (at 132.08 130.81 0))
+    (property "Footprint" "" (id 2) (at 132.08 125.73 0)
+      (effects (font (size 1.27 1.27)) hide)
+    )
+    (property "Datasheet" "" (id 3) (at 132.08 125.73 0)
+      (effects (font (size 1.27 1.27)) hide)
+    )
+    (pin "1")
+  )
+  (symbol (lib_id "Homssymbols:CANbus") (at 69.85 149.86 0) (unit 1)
+    (in_bom yes) (on_board yes) (fields_autoplaced)
+    (property "Reference" "U?" (id 0) (at 90.17 132.08 0))
+    (property "Value" "CANbus" (id 1) (at 90.17 134.62 0))
+    (property "Footprint" "" (id 2) (at 76.2 144.78 0)
+      (effects (font (size 1.27 1.27)) hide)
+    )
+    (property "Datasheet" "" (id 3) (at 76.2 144.78 0)
+      (effects (font (size 1.27 1.27)) hide)
+    )
+    (pin "")
+    (pin "")
+    (pin "")
+    (pin "")
+    (pin "")
+    (pin "")
+    (pin "")
+    (pin "")
+    (pin "")
   )
   (symbol (lib_id "Homssymbols:TI_J1{slash}J3") (at 106.68 115.57 0) (unit 1)

Commit message: motor update
added the motor wiring to the tractive system
Connections:
- new net: U?. (GND), U?. (To_TI_CAN_L) (x2)

Commit message: 2/15
Connections:
- new net: U?. (GND), U?. (To_TI_CAN_L) (x2)

Commit message: keyswitch
updated key switch to be pin 6. did other things
Connections:
- new net: U?. (GND), U?. (To_TI_CAN_L) (x2)

Commit message: Added Keyswitch Relay & 12V battery
Connections:
- new net: U?. (GND), U?. (To_TI_CAN_L) (x2)

Commit message: fixed throttle wiring
removed throttle resistor and wired throttle pins 2 and 4 together
Connections:
- new net: U?. (GND), U?. (To_TI_CAN_L) (x2)
Changed lines of the file:
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@@
 (kicad_sch (version 20211123) (generator eeschema)
   (paper "A")
+  (title_block
+    (date "2023-02-28")
+  )
   (wire (pts (xy 137.16 140.97) (xy 137.16 125.73))
     (stroke (width 0) (type default) (color 0 0 0 0))
