File: KiCad/NR23_Schematic_v1.0/DriverInterface.kicad_sch (KiCad schematic)
At the start: 0 parts

Commit message: microcontroller + symbol library
Parts:
- added U?: Dash, symbol Homssymbols:Dash
Connections:
- new net CAN_H_DASH: U?. (GND)
Changed lines of the file:
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@@
 (kicad_sch (version 20211123) (generator eeschema)
   (paper "A")
+  (wire (pts (xy 85.09 50.8) (xy 92.71 50.8))
+    (stroke (width 0) (type default) (color 0 0 0 0))
+  )
   (text "The throttle pedal is now inside the tractive system schematic"
     (at 81.28 99.06 0)
     (effects (font (size 3 3)) (justify left bottom))
   )
+  (hierarchical_label "CAN_H_DASH" (shape input) (at 92.71 50.8 0)
+    (effects (font (size 1.27 1.27)) (justify left))
+  )
+  (symbol (lib_id "Homssymbols:Dash") (at 62.23 67.31 0) (unit 1)
+    (in_bom yes) (on_board yes) (fields_autoplaced)
+    (property "Reference" "U?" (id 0) (at 76.2 41.91 0))
+    (property "Value" "Dash" (id 1) (at 76.2 44.45 0))
+    (property "Footprint" "" (id 2) (at 62.23 67.31 0)
+      (effects (font (size 1.27 1.27)) hide)
+    )
+    (property "Datasheet" "" (id 3) (at 62.23 67.31 0)
+      (effects (font (size 1.27 1.27)) hide)
+    )
+    (pin "")
+    (pin "")
+    (pin "")
+  )
 )

Commit message: end of class 2/13
Connections:
- net CAN_H_DASH is gone; now on net CANBus_dash_L: U?. (GND)
- net CANBus_dash_L: now reaches U?. (GND)
- new net CANBus_dash_H: U?. (GND)
Changed lines of the file:
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@@
+    (stroke (width 0) (type default) (color 0 0 0 0))
+  )
+  (wire (pts (xy 85.09 55.88) (xy 92.71 55.88))
+    (stroke (width 0) (type default) (color 0 0 0 0))
+  )
+  (wire (pts (xy 85.09 53.34) (xy 92.71 53.34))
     (stroke (width 0) (type default) (color 0 0 0 0))
   )
@@
     (effects (font (size 3 3)) (justify left bottom))
   )
-  (hierarchical_label "CAN_H_DASH" (shape input) (at 92.71 50.8 0)
+  (hierarchical_label "CANBus_dash_L" (shape input) (at 92.71 53.34 0)
     (effects (font (size 1.27 1.27)) (justify left))
   )
+  (hierarchical_label "CANBus_dash_H" (shape input) (at 92.71 50.8 0)
+    (effects (font (size 1.27 1.27)) (justify left))
+  )
