File: KiCad/NR23_Schematic_v1.0/BenchTop.kicad_sch (KiCad schematic)
At the start: 13 parts, among them M1 Zero_7R_Motor

Commit message: start of class 18APR23
Connections:
- net at U?. (M3): now also J?.2 (Pin_2), J?.4 (Pin_4)

Commit message: start of class 26apr23
Connections:
- net at U?. (M3): now also J?.2 (Pin_2), J?.4 (Pin_4)

Commit message: endof day 26APR23
changed the wires going into the ti board box in order to match what is actually on the car
Connections:
- net at U?. (M3): now also J?.2 (Pin_2), J?.4 (Pin_4)

Commit message: end of class on 01APR23 - battery stuff
Added new battery connections and reprinted battery schematic
Connections:
- net at U?. (M3): now also J?.2 (Pin_2), J?.4 (Pin_4)

Commit message: end of day 02APR23
Connections:
- net at U?. (M3): now also J?.2 (Pin_2), J?.4 (Pin_4)

Commit message: reee
Connections:
- net at U?. (M3): now also J?.2 (Pin_2), J?.4 (Pin_4)
Changed lines of the file:
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@@
   (title_block
     (title "Tractive System")
-    (date "2023-03-03")
+    (date "2023-05-03")
   )
   (junction (at 133.35 95.25) (diameter 0) (color 0 0 0 0)

Commit message: Base update (V3)
Connections:
- net at U?. (M3): now also J?.2 (Pin_2), J?.4 (Pin_4)
