File: KiCad/NR23_Schematic_v1.0/NR23_Schematic_v1.0.kicad_sch (KiCad schematic)
At the start: 0 parts

Commit message: end of day 05APR23
Other:
- removed sheet Microcontroller
Changed lines of the file:
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@@
 (kicad_sch (version 20211123) (generator eeschema)
-  (paper "A")
+  (paper "User" 334.01 216.002)
   (title_block
     (date "2023-04-04")
@@
     )
   )
-  (sheet (at 106.68 160.02) (size 49.53 30.48)
-    (stroke (width 0.1524) (type solid) (color 0 0 0 0))
-    (fill (color 0 0 0 0.0000))
-    (property "Sheet name" "Microcontroller" (id 0) (at 105.41 158.75 0)
-      (effects (font (size 5 5)) (justify left bottom))
-    )
-    (property "Sheet file" "Microcontroller.kicad_sch" (id 1) (at 106.68 172.72 0)
-      (effects (font (size 1.27 1.27)) (justify left top))
-    )
-  )
   (sheet_instances
     (path "/" (page "1"))
     (path "/8302703f-65d0-4b91-aeea-6f721ab57e4c" (page "1"))
-    (path "/c7466bb0-ebde-4ea4-90e3-94511e3895a3" (page "2"))
     (path "/16ced548-a4c4-4a05-b722-8e9610f878cc" (page "5"))
+    (path "/8302703f-65d0-4b91-aeea-6f721ab57e4c/97abb871-5579-4630-a10b-2cee2773b5bb" (page "6"))
     (path "/6b38ef1b-89ba-46d1-8032-b895c26a5218" (page "7"))
   )
   (symbol_instances
-    (path "/c7466bb0-ebde-4ea4-90e3-94511e3895a3/abd2a7f6-194b-4f90-9352-cc86eaabf27b"
+    (path "/8302703f-65d0-4b91-aeea-6f721ab57e4c/97abb871-5579-4630-a10b-2cee2773b5bb/abd2a7f6-194b-4f90-9352-cc86eaabf27b"
       (reference "#PWR?") (unit 1) (value "GND") (footprint "")
     )
-    (path "/c7466bb0-ebde-4ea4-90e3-94511e3895a3/aefa985d-2a08-4349-90af-e8fd54a309c3"
+    (path "/8302703f-65d0-4b91-aeea-6f721ab57e4c/97abb871-5579-4630-a10b-2cee2773b5bb/aefa985d-2a08-4349-90af-e8fd54a309c3"
       (reference "#PWR?") (unit 1) (value "GND") (footprint "")
     )
@@
       (reference "BT?") (unit 1) (value "7.2KW_Battery") (footprint "")
     )
-    (path "/8302703f-65d0-4b91-aeea-6f721ab57e4c/9ec1d7fc-6f5f-41a1-a450-d625e8c70d57"
+    (path "/8302703f-65d0-4b91-aeea-6f721ab57e4c/39d10f1e-0e39-4617-84d3-0f39768316a5"
       (reference "BTaux") (unit 1) (value "12V") (footprint "")
     )
@@
       (reference "BTmain") (unit 1) (value "7.2KW_BatteryALLPINS") (footprint "")
     )
-    (path "/8302703f-65d0-4b91-aeea-6f721ab57e4c/ba497376-f3b3-4aa7-8c24-837b232c4c3d"
+    (path "/8302703f-65d0-4b91-aeea-6f721ab57e4c/0ff0a299-f28e-4254-8f91-d87a10b36f6c"
       (reference "F?") (unit 1) (value "Sevcon Fuse") (footprint "")
     )
@@
       (reference "F?") (unit 1) (value "Fuse") (footprint "")
     )
+    (path "/8302703f-65d0-4b91-aeea-6f721ab57e4c/97abb871-5579-4630-a10b-2cee2773b5bb/1dd5ea95-d588-470f-9d97-474e57890a75"
+      (reference "J?") (unit 1) (value "Display Connection") (footprint "")
+    )
+    (path "/8302703f-65d0-4b91-aeea-6f721ab57e4c/216444df-625d-4820-8680-e1f7fefb27ea"
+      (reference "J?") (unit 1) (value "Deutsch") (footprint "")
+    )
     (path "/8302703f-65d0-4b91-aeea-6f721ab57e4c/29343fe7-1090-4f39-b166-f0431019621b"
       (reference "J?") (unit 1) (value "Dash TI Connection") (footprint "")
     )
+    (path "/8302703f-65d0-4b91-aeea-6f721ab57e4c/97abb871-5579-4630-a10b-2cee2773b5bb/2a7f9b9a-014a-459c-9a52-e32d8d4a03ec"
+      (reference "J?") (unit 1) (value "Dash TI Connection") (footprint "")
+    )
     (path "/8302703f-65d0-4b91-aeea-6f721ab57e4c/33462402-8cb3-4f96-960d-15ae2e14504f"
       (reference "J?") (unit 1) (value "CAN Connector") (footprint "")
@@
       (reference "J?") (unit 1) (value "M_con") (footprint "")
     )
+    (path "/8302703f-65d0-4b91-aeea-6f721ab57e4c/97abb871-5579-4630-a10b-2cee2773b5bb/819680fd-28b0-4f33-88c0-dda0b2179bd1"
+      (reference "J?") (unit 1) (value "CAN Connector") (footprint "")
+    )
     (path "/8302703f-65d0-4b91-aeea-6f721ab57e4c/91ff6b73-349d-49e4-9742-09d502f987be"
       (reference "J?") (unit 1) (value "Deutsch") (footprint "")
@@
       (reference "J?") (unit 1) (value "F_con") (footprint "")
     )
-    (path "/8302703f-65d0-4b91-aeea-6f721ab57e4c/de29f7ed-664a-479e-9fdb-f102e88408fb"
-      (reference "J?") (unit 1) (value "Deutsch") (footprint "")
-    )
     (path "/6b38ef1b-89ba-46d1-8032-b895c26a5218/de29f7ed-664a-479e-9fdb-f102e88408fb"
       (reference "J?") (unit 1) (value "M_con") (footprint "")
@@
       (reference "K?") (unit 1) (value "Key Switch Relay") (footprint "Relay_THT:Relay_1P1T_NO_10x24x18.8mm_Panasonic_ADW11xxxxW_THT")
     )
-    (path "/8302703f-65d0-4b91-aeea-6f721ab57e4c/91be2d7e-1603-4ffc-85db-9cef433a5348"
+    (path "/8302703f-65d0-4b91-aeea-6f721ab57e4c/a93530ce-8b22-4b63-b724-6c1e4d5cd8be"
+      (reference "K?") (unit 1) (value "Line Contactor") (footprint "Relay_THT:Relay_1P1T_NO_10x24x18.8mm_Panasonic_ADW11xxxxW_THT")
+    )
+    (path "/8302703f-65d0-4b91-aeea-6f721ab57e4c/a9e985c1-5127-467f-ba30-fc49c207bd55"
       (reference "K?") (unit 1) (value "Key Switch Relay") (footprint "Relay_THT:Relay_1P1T_NO_10x24x18.8mm_Panasonic_ADW11xxxxW_THT")
     )
@@
       (reference "K?") (unit 1) (value "Line Contactor") (footprint "Relay_THT:Relay_1P1T_NO_10x24x18.8mm_Panasonic_ADW11xxxxW_THT")
     )
-    (path "/8302703f-65d0-4b91-aeea-6f721ab57e4c/b190c8cb-bd8a-4856-a017-7c47d784415d"
-      (reference "K?") (unit 1) (value "Line Contactor") (footprint "Relay_THT:Relay_1P1T_NO_10x24x18.8mm_Panasonic_ADW11xxxxW_THT")
-    )
     (path "/8302703f-65d0-4b91-aeea-6f721ab57e4c/35fc9197-f5a2-4771-8459-3e635ee3ee3c"
       (reference "LA1") (unit 1) (value "TI power Light") (footprint "")
@@
       (reference "LA5") (unit 1) (value "REV/N Light") (footprint "")
     )
-    (path "/8302703f-65d0-4b91-aeea-6f721ab57e4c/17f5dc4f-ba2e-4459-9469-5c2da575d700"
+    (path "/8302703f-65d0-4b91-aeea-6f721ab57e4c/133ace85-6439-4feb-9413-75f9037bf88e"
       (reference "M1") (unit 1) (value "Zero_7R_Motor") (footprint "")
     )
@@
       (reference "SW?") (unit 1) (value "Shifter Switch") (footprint "")
     )
-    (path "/8302703f-65d0-4b91-aeea-6f721ab57e4c/839a2160-4be7-4a71-b4f3-e2d027441525"
-      (reference "SW?") (unit 1) (value "HV Safety Switch (behind driver)") (footprint "")
-    )
     (path "/6b38ef1b-89ba-46d1-8032-b895c26a5218/839a2160-4be7-4a71-b4f3-e2d027441525"
       (reference "SW?") (unit 1) (value "HV Safety Switch") (footprint "")
@@
       (reference "SW?") (unit 1) (value "100V E-stop (Left)") (footprint "")
     )
+    (path "/8302703f-65d0-4b91-aeea-6f721ab57e4c/c3efaf65-8006-4868-9f6d-0b34664fb679"
+      (reference "SW?") (unit 1) (value "HV Safety Switch (behind driver)") (footprint "")
+    )
     (path "/8302703f-65d0-4b91-aeea-6f721ab57e4c/c61cd80c-144e-4e2a-b98d-2afd10895cc1"
       (reference "SW?") (unit 1) (value "100V E-stop (Right)") (footprint "")
@@
       (reference "U?") (unit 1) (value "Throttle") (footprint "")
     )
-    (path "/8302703f-65d0-4b91-aeea-6f721ab57e4c/0aa54167-f3d9-467b-bc69-db1827651c6c"
+    (path "/8302703f-65d0-4b91-aeea-6f721ab57e4c/0e1a68e2-749f-4c4a-963e-7ad1987b1071"
       (reference "U?") (unit 1) (value "Throttle") (footprint "")
-    )
-    (path "/8302703f-65d0-4b91-aeea-6f721ab57e4c/35333229-0e5e-47a2-bb43-fcfbf8fd658d"
-      (reference "U?") (unit 1) (value "Sevcon_Gen4_Size6") (footprint "")
     )
     (path "/6b38ef1b-89ba-46d1-8032-b895c26a5218/35333229-0e5e-47a2-bb43-fcfbf8fd658d"
       (reference "U?") (unit 1) (value "Sevcon_Gen4_Size6") (footprint "")
     )
-    (path "/c7466bb0-ebde-4ea4-90e3-94511e3895a3/699a947b-7503-4a2e-aeca-27dd918b3280"
+    (path "/8302703f-65d0-4b91-aeea-6f721ab57e4c/97abb871-5579-4630-a10b-2cee2773b5bb/699a947b-7503-4a2e-aeca-27dd918b3280"
       (reference "U?") (unit 1) (value "TI_J12_CANbus") (footprint "")
+    )
+    (path "/8302703f-65d0-4b91-aeea-6f721ab57e4c/86d607a7-2b22-494c-98f1-8e82fb114d95"
+      (reference "U?") (unit 1) (value "Sevcon_Gen4_Size6") (footprint "")
     )
     (path "/16ced548-a4c4-4a05-b722-8e9610f878cc/942b0a04-1bf0-4324-8c6e-417346d8e5d0"
       (reference "U?") (unit 1) (value "xbee") (footprint "")
     )
-    (path "/c7466bb0-ebde-4ea4-90e3-94511e3895a3/991d9159-ee3b-4883-9868-58693594f778"
+    (path "/8302703f-65d0-4b91-aeea-6f721ab57e4c/97abb871-5579-4630-a10b-2cee2773b5bb/991d9159-ee3b-4883-9868-58693594f778"
       (reference "U?") (unit 1) (value "TI_Board") (footprint "")
     )
-    (path "/c7466bb0-ebde-4ea4-90e3-94511e3895a3/c4d2efd0-b388-45fb-bba7-22b5c621151d"
+    (path "/8302703f-65d0-4b91-aeea-6f721ab57e4c/97abb871-5579-4630-a10b-2cee2773b5bb/c4d2efd0-b388-45fb-bba7-22b5c621151d"
       (reference "U?") (unit 1) (value "CANbus") (footprint "")
     )
-    (path "/c7466bb0-ebde-4ea4-90e3-94511e3895a3/dd05f672-8c08-4b2b-9bb3-8f78a97dab20"
+    (path "/8302703f-65d0-4b91-aeea-6f721ab57e4c/97abb871-5579-4630-a10b-2cee2773b5bb/dd05f672-8c08-4b2b-9bb3-8f78a97dab20"
       (reference "U?") (unit 1) (value "TI_J1/J3") (footprint "")
     )

Commit message: start of class 18APR23
Changed lines of the file:
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@@
     (date "2023-04-04")
   )
-  (sheet (at 26.67 156.21) (size 50.8 38.1)
+  (sheet (at 39.37 132.08) (size 115.57 64.77)
     (stroke (width 0.1524) (type solid) (color 0 0 0 0))
     (fill (color 0 0 0 0.0000))
-    (property "Sheet name" "Telemetry" (id 0) (at 26.67 153.67 0)
+    (property "Sheet name" "Telemetry" (id 0) (at 39.37 129.54 0)
       (effects (font (size 5 5)) (justify left bottom))
     )
-    (property "Sheet file" "Telemetry.kicad_sch" (id 1) (at 26.67 194.8946 0)
+    (property "Sheet file" "Telemetry.kicad_sch" (id 1) (at 39.37 170.7646 0)
       (effects (font (size 1.27 1.27)) (justify left top))
     )
   )
-  (sheet (at 195.58 132.08) (size 59.69 39.37) (fields_autoplaced)
+  (sheet (at 195.58 132.08) (size 110.49 35.56) (fields_autoplaced)
     (stroke (width 0.1524) (type solid) (color 0 0 0 0))
     (fill (color 0 0 0 0.0000))
@@
       (effects (font (size 5 5)) (justify left bottom))
     )
-    (property "Sheet file" "BenchTop.kicad_sch" (id 1) (at 195.58 172.0346 0)
+    (property "Sheet file" "BenchTop.kicad_sch" (id 1) (at 195.58 168.2246 0)
       (effects (font (size 1.27 1.27)) (justify left top))
     )
@@
   )
   (symbol_instances
+    (path "/8302703f-65d0-4b91-aeea-6f721ab57e4c/97abb871-5579-4630-a10b-2cee2773b5bb/0cc246a4-8870-49dd-945c-fbfffb55b703"
+      (reference "#PWR?") (unit 1) (value "GND") (footprint "")
+    )
+    (path "/8302703f-65d0-4b91-aeea-6f721ab57e4c/97abb871-5579-4630-a10b-2cee2773b5bb/5b678e11-7d21-49c7-87bd-7953081d7748"
+      (reference "#PWR?") (unit 1) (value "GND") (footprint "")
+    )
+    (path "/8302703f-65d0-4b91-aeea-6f721ab57e4c/97abb871-5579-4630-a10b-2cee2773b5bb/86242390-ce71-4a1c-a74a-66c29943dff8"
+      (reference "#PWR?") (unit 1) (value "GND") (footprint "")
+    )
+    (path "/8302703f-65d0-4b91-aeea-6f721ab57e4c/97abb871-5579-4630-a10b-2cee2773b5bb/934055cb-9d39-4ad1-ae76-261d73ee61b7"
+      (reference "#PWR?") (unit 1) (value "GND") (footprint "")
+    )
+    (path "/8302703f-65d0-4b91-aeea-6f721ab57e4c/97abb871-5579-4630-a10b-2cee2773b5bb/a095cb59-e422-4afa-939f-01dc6aa5dd91"
+      (reference "#PWR?") (unit 1) (value "GND") (footprint "")
+    )
     (path "/8302703f-65d0-4b91-aeea-6f721ab57e4c/97abb871-5579-4630-a10b-2cee2773b5bb/abd2a7f6-194b-4f90-9352-cc86eaabf27b"
       (reference "#PWR?") (unit 1) (value "GND") (footprint "")
     )
     (path "/8302703f-65d0-4b91-aeea-6f721ab57e4c/97abb871-5579-4630-a10b-2cee2773b5bb/aefa985d-2a08-4349-90af-e8fd54a309c3"
+      (reference "#PWR?") (unit 1) (value "GND") (footprint "")
+    )
+    (path "/8302703f-65d0-4b91-aeea-6f721ab57e4c/97abb871-5579-4630-a10b-2cee2773b5bb/b105d02e-5b3f-492d-b9d6-bccabd476c30"
       (reference "#PWR?") (unit 1) (value "GND") (footprint "")
     )
@@
       (reference "BTmain") (unit 1) (value "7.2KW_BatteryALLPINS") (footprint "")
     )
+    (path "/8302703f-65d0-4b91-aeea-6f721ab57e4c/97abb871-5579-4630-a10b-2cee2773b5bb/33edf8a8-a3e4-48e9-80f7-6f14e9047a71"
+      (reference "D?") (unit 1) (value "D") (footprint "")
+    )
+    (path "/8302703f-65d0-4b91-aeea-6f721ab57e4c/97abb871-5579-4630-a10b-2cee2773b5bb/3dd41065-0661-4611-b751-7b7457dab073"
+      (reference "D?") (unit 1) (value "D") (footprint "")
+    )
+    (path "/8302703f-65d0-4b91-aeea-6f721ab57e4c/97abb871-5579-4630-a10b-2cee2773b5bb/cb3f31f3-7647-4909-937e-3d544217c1ef"
+      (reference "D?") (unit 1) (value "D") (footprint "")
+    )
     (path "/8302703f-65d0-4b91-aeea-6f721ab57e4c/0ff0a299-f28e-4254-8f91-d87a10b36f6c"
       (reference "F?") (unit 1) (value "Sevcon Fuse") (footprint "")
@@
       (reference "F?") (unit 1) (value "Fuse") (footprint "")
     )
+    (path "/8302703f-65d0-4b91-aeea-6f721ab57e4c/c3efaf65-8006-4868-9f6d-0b34664fb679"
+      (reference "HVSS") (unit 1) (value "HV Safety Switch (behind driver)") (footprint "")
+    )
     (path "/8302703f-65d0-4b91-aeea-6f721ab57e4c/97abb871-5579-4630-a10b-2cee2773b5bb/1dd5ea95-d588-470f-9d97-474e57890a75"
       (reference "J?") (unit 1) (value "Display Connection") (footprint "")
@@
       (reference "J?") (unit 1) (value "Dash Key Switch Connection") (footprint "")
     )
-    (path "/8302703f-65d0-4b91-aeea-6f721ab57e4c/4f7773d6-0ce1-4de2-b33c-40a7545a2a6c"
-      (reference "J?") (unit 1) (value "Dash 12 power connection") (footprint "")
-    )
     (path "/8302703f-65d0-4b91-aeea-6f721ab57e4c/677d3ecc-41bd-42e2-8c0e-9eee2eeadf6d"
       (reference "J?") (unit 1) (value "Alt Dash 12 power connection") (footprint "")
@@
       (reference "M1") (unit 1) (value "Zero_7R_Motor") (footprint "")
     )
+    (path "/8302703f-65d0-4b91-aeea-6f721ab57e4c/97abb871-5579-4630-a10b-2cee2773b5bb/4cfe98f9-aa78-4658-9e93-07cade6de232"
+      (reference "Q?") (unit 1) (value "Q_NMOS_DGS") (footprint "")
+    )
+    (path "/8302703f-65d0-4b91-aeea-6f721ab57e4c/97abb871-5579-4630-a10b-2cee2773b5bb/d68c45a5-3fdd-4a29-9ea0-4fa67786e0ef"
+      (reference "Q?") (unit 1) (value "Q_NMOS_DGS") (footprint "")
+    )
+    (path "/8302703f-65d0-4b91-aeea-6f721ab57e4c/97abb871-5579-4630-a10b-2cee2773b5bb/faf03bf7-4254-4b9f-b70e-e4b84b8615c6"
+      (reference "Q?") (unit 1) (value "Q_NMOS_DGS") (footprint "")
+    )
+    (path "/8302703f-65d0-4b91-aeea-6f721ab57e4c/97abb871-5579-4630-a10b-2cee2773b5bb/2d9cf3fe-accd-4c59-87b2-dbf79ebc59cd"
+      (reference "R?") (unit 1) (value "R_US") (footprint "")
+    )
+    (path "/8302703f-65d0-4b91-aeea-6f721ab57e4c/97abb871-5579-4630-a10b-2cee2773b5bb/610df3be-18c0-42b0-9161-50b370e0205d"
+      (reference "R?") (unit 1) (value "R_US") (footprint "")
+    )
+    (path "/8302703f-65d0-4b91-aeea-6f721ab57e4c/97abb871-5579-4630-a10b-2cee2773b5bb/6917848f-da8c-4c38-8fa7-5aa80b3bfb19"
+      (reference "R?") (unit 1) (value "R_US") (footprint "")
+    )
+    (path "/8302703f-65d0-4b91-aeea-6f721ab57e4c/97abb871-5579-4630-a10b-2cee2773b5bb/abdb6156-d278-4176-813d-88b3fac1714c"
+      (reference "R?") (unit 1) (value "R_US") (footprint "")
+    )
+    (path "/8302703f-65d0-4b91-aeea-6f721ab57e4c/97abb871-5579-4630-a10b-2cee2773b5bb/c074acdc-73b0-49e5-a95e-d94754a448e2"
+      (reference "R?") (unit 1) (value "R_US") (footprint "")
+    )
+    (path "/8302703f-65d0-4b91-aeea-6f721ab57e4c/97abb871-5579-4630-a10b-2cee2773b5bb/c63e61ff-1cf3-4748-b8bd-e010cc68eeca"
+      (reference "R?") (unit 1) (value "R_US") (footprint "")
+    )
     (path "/8302703f-65d0-4b91-aeea-6f721ab57e4c/3c4e7487-ab0a-423b-bce9-bfd53c73f666"
       (reference "SW?") (unit 1) (value "Key Switch") (footprint "")
@@
       (reference "SW?") (unit 1) (value "100V E-stop (Left)") (footprint "")
     )
-    (path "/8302703f-65d0-4b91-aeea-6f721ab57e4c/c3efaf65-8006-4868-9f6d-0b34664fb679"
-      (reference "SW?") (unit 1) (value "HV Safety Switch (behind driver)") (footprint "")
-    )
     (path "/8302703f-65d0-4b91-aeea-6f721ab57e4c/c61cd80c-144e-4e2a-b98d-2afd10895cc1"
