File: KiCad/NR23_Schematic_v1.0/TractiveSystem.kicad_sch (KiCad schematic)
At the start: 29 parts, among them J1 M_con, J2 F_con, J3 Dash power connection, J4 Dash power connection, J5 Dash TI Connection, J6 Deutsch, J7 Deutsch, J8 CAN Connector, K1 Line Contactor, K2 Key Switch Relay, M1 Zero_7R_Motor, SW1 TI power switch, SW2 Shifter Switch, SW3 100V E-stop (Right), SW4 100V E-stop (Left), SW5 Key Switch, SW6 12V E-stop, U1 Sevcon_Gen4_Size6, U2 Throttle

Commit message: reee
Parts:
- BTaux1: value 20V -> 12V
Connections:
- net B-: now also BTaux1.2 (-), J4.4 (Pin_4)
- net system_on_fromBattery: now also J8.7 (Pin_7)
- net throttle_en_fromBattery: now also J8.6 (Pin_6)
- no-connect marks 23 -> 21
Other:
- note added: "<- Hole in TI box for the CAN connections"
- note added: "ABC or ACB"
- note added: "ADD HV ACTIVE LIGHT HERE ^"
- note added: "Hole in TI box for the dash connections ->"
- note added: "throttle_en and system_on connected to 5V off of the TI board (~20mA)"
- note removed: "? Are we in ABC or ACB?"
- note removed: "NEED HV ACTIVE LIGHT HERE ^"
- note removed: "One hole in TI box -> for the CAN connections"
- note removed: "Two holes in TI box for the dash connections ->"
Changed lines of the file:
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@@
   (title_block
     (title "Tractive System")
-    (date "2023-04-05")
+    (date "2023-05-03")
     (rev "Print 1")
   )
   (junction (at 49.53 40.64) (diameter 0) (color 0 0 0 0)
   )
+  (junction (at 127 87.63) (diameter 0) (color 0 0 0 0)
+  )
   (junction (at 121.92 121.92) (diameter 0) (color 0 0 0 0)
   )
   (junction (at 46.99 27.94) (diameter 0) (color 0 0 0 0)
   )
+  (junction (at 175.26 151.13) (diameter 0) (color 0 0 0 0)
+  )
   (junction (at 270.51 133.35) (diameter 0) (color 0 0 0 0)
   )
@@
   (junction (at 175.26 105.41) (diameter 0) (color 0 0 0 0)
   )
-  (no_connect (at 259.08 78.74))
   (no_connect (at 71.12 113.03))
   (no_connect (at 74.93 165.1))
@@
   (no_connect (at 127 60.96))
   (no_connect (at 31.75 152.4))
-  (no_connect (at 271.78 78.74))
   (no_connect (at 80.01 175.26))
   (no_connect (at 265.43 143.51))
@@
     (stroke (width 0) (type default) (color 0 0 0 0))
   )
-  (wire (pts (xy 172.72 151.13) (xy 177.8 151.13))
+  (wire (pts (xy 172.72 151.13) (xy 175.26 151.13))
     (stroke (width 0) (type default) (color 0 0 0 0))
   )
@@
     (stroke (width 0.5) (type default) (color 0 0 0 0))
   )
+  (wire (pts (xy 138.43 87.63) (xy 127 87.63))
+    (stroke (width 0) (type default) (color 0 0 0 0))
+  )
   (bus (pts (xy 81.28 50.8) (xy 81.28 54.61))
     (stroke (width 0) (type default) (color 0 0 0 0))
@@
     (stroke (width 0) (type default) (color 0 0 0 0))
   )
+  (wire (pts (xy 175.26 151.13) (xy 177.8 151.13))
+    (stroke (width 0) (type default) (color 0 0 0 0))
+  )
   (polyline (pts (xy 157.48 168.91) (xy 157.48 168.91))
     (stroke (width 0.5) (type default) (color 0 0 0 0))
@@
     (stroke (width 0.5) (type solid) (color 0 0 0 0))
   )
+  (wire (pts (xy 138.43 161.29) (xy 175.26 161.29))
+    (stroke (width 0) (type default) (color 0 0 0 0))
+  )
   (polyline (pts (xy 297.18 54.61) (xy 162.56 54.61))
     (stroke (width 0.75) (type solid) (color 0 0 0 0))
@@
   )
   (wire (pts (xy 116.84 59.69) (xy 116.84 60.96))
+    (stroke (width 0) (type default) (color 0 0 0 0))
+  )
+  (wire (pts (xy 138.43 87.63) (xy 138.43 161.29))
     (stroke (width 0) (type default) (color 0 0 0 0))
   )
@@
     (stroke (width 0.5) (type default) (color 0 0 0 0))
   )
-  (text "Two holes in TI box for\nthe dash connections ->" (at 135.89 53.34 0)
+  (wire (pts (xy 175.26 161.29) (xy 175.26 151.13))
+    (stroke (width 0) (type default) (color 0 0 0 0))
+  )
+  (text "Hole in TI box for\nthe dash connections ->" (at 137.16 53.34 0)
     (effects (font (size 1.27 1.27)) (justify left bottom))
   )
@@
   )
   (text "Fuse is not installed\nbut could be installed\nin this location"
-    (at 118.11 134.62 0)
+    (at 110.49 134.62 0)
     (effects (font (size 1.5 1.5)) (justify left bottom))
   )
@@
     (effects (font (size 1.27 1.27)) (justify left bottom))
   )
-  (text "NEED HV ACTIVE LIGHT HERE ^" (at 90.17 123.19 180)
+  (text "ADD HV ACTIVE LIGHT HERE ^" (at 90.17 123.19 180)
     (effects (font (size 1.27 1.27) (thickness 0.254) bold italic) (justify right bottom))
   )
@@
     (effects (font (size 1.27 1.27)) (justify left bottom))
   )
-  (text "One hole in TI box ->\nfor the CAN connections" (at 303.53 76.2 0)
+  (text "<- Hole in TI box for\nthe CAN connections" (at 299.72 57.15 0)
+    (effects (font (size 1.27 1.27)) (justify left bottom))
+  )
+  (text "throttle_en and system_on\nconnected to 5V off of the\nTI board (~20mA)"
+    (at 254 90.17 0)
     (effects (font (size 1.27 1.27)) (justify left bottom))
   )
@@
     (effects (font (size 1.75 1.75) (thickness 0.35) bold) (justify left bottom))
   )
-  (text "? Are we in ABC or ACB?" (at 153.67 200.66 0)
-    (effects (font (size 1.75 1.75) bold italic) (justify left bottom))
+  (text "ABC or ACB" (at 154.94 196.85 0)
+    (effects (font (size 1.75 1.75)) (justify left bottom))
   )
   (label "EnA" (at 172.72 128.27 0)
@@
   )
   (label "throttle_en" (at 21.59 109.22 90)
+    (effects (font (size 1.27 1.27)) (justify left bottom))
+  )
+  (label "Common Battery Ground" (at 137.16 87.63 0)
     (effects (font (size 1.27 1.27)) (justify left bottom))
   )
@@
   )
   (label "Line Contactor (Cont1)" (at 91.44 105.41 0)
+    (effects (font (size 1.27 1.27)) (justify left bottom))
+  )
+  (label "Common Battery Ground" (at 138.43 151.13 90)
     (effects (font (size 1.27 1.27)) (justify left bottom))
   )
@@
     )
   )
-  (global_label "system_on_fromBattery" (shape input) (at 270.51 86.36 0) (fields_autoplaced)
-    (effects (font (size 1.27 1.27) (thickness 0.254) bold) (justify left))
-    (property "Intersheet References" "${INTERSHEET_REFS}" (id 0) (at 294.9454 86.233 0)
-      (effects (font (size 1.27 1.27) (thickness 0.254) bold) (justify left) hide)
+  (global_label "system_on_fromBattery" (shape input) (at 259.08 78.74 180) (fields_autoplaced)
+    (effects (font (size 1.27 1.27) (thickness 0.254) bold) (justify right))
+    (property "Intersheet References" "${INTERSHEET_REFS}" (id 0) (at 234.6446 78.867 0)
+      (effects (font (size 1.27 1.27) (thickness 0.254) bold) (justify right) hide)
     )
   )
@@
     )
   )
-  (global_label "throttle_en_fromBattery" (shape input) (at 262.89 91.44 0) (fields_autoplaced)
-    (effects (font (size 1.27 1.27) (thickness 0.254) bold) (justify left))
-    (property "Intersheet References" "${INTERSHEET_REFS}" (id 0) (at 287.7487 91.313 0)
+  (global_label "throttle_en_fromBattery" (shape input) (at 271.78 78.74 0) (fields_autoplaced)
+    (effects (font (size 1.27 1.27) (thickness 0.254) bold) (justify left))
+    (property "Intersheet References" "${INTERSHEET_REFS}" (id 0) (at 296.6387 78.613 0)
       (effects (font (size 1.27 1.27) (thickness 0.254) bold) (justify left) hide)
     )
@@
       (effects (font (size 1.27 1.27)) (justify right))
     )
-    (property "Value" "CAN Connector" (id 1) (at 259.08 82.55 0)
+    (property "Value" "CAN Connector" (id 1) (at 257.81 82.55 0)
       (effects (font (size 1.27 1.27)) (justify right))
     )
@@
       (effects (font (size 1.27 1.27)) (justify left))
     )
-    (property "Value" "20V" (id 1) (at 132.08 85.09 90)
+    (property "Value" "12V" (id 1) (at 132.08 85.09 90)
       (effects (font (size 1.27 1.27)) (justify left))
     )

Commit message: Base update (V3)
Parts:
- added J9: XBI, symbol Connector_Generic:Conn_02x06_Counter_Clockwise
Other:
- removed sheet NSWC Battery Wiring
- note removed: "CLICK HERE ^ TO SEE HOW NSWC CRANE WIRED THEIR LONGBRICK"
- note removed: "FS1 Pedal pressed: logic 1 Pedal static: logic 0"
- note removed: "Fuse is not installed but could be installed in this location"
- note removed: "Harness 1: Sevcon to Footwell"
- note removed: "The chassis isolation pin is attached to the frame via a ring terminal on one of the Sevcon heatsink bolts"
- note removed: "This throttle is not FSAE compliant in this design."
- note removed: "Three large power wires to the motor"
- moved on the sheet: H1
