File: KiCad/Car_TractiveSystem_v2.kicad_sch (KiCad schematic)
At the start: 26 parts, among them J1 M_con, J2 F_con, J5 Dash TI Connection, J6 Deutsch, J7 Deutsch, J8 CAN Connector, K1 Line Contactor, K2 Key Switch Relay, M1 Zero_7R_Motor, SW1 TI power switch, SW2 Shifter Switch, SW3 100V E-stop (Right), SW4 100V E-stop (Left), SW5 Key Switch, SW6 12V E-stop, U1 Sevcon_Gen4_Size6, U2 Throttle

Commit message: 24OCT23
Changed lines of the file:
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@@
     (stroke (width 0) (type default))
   )
-  (bus_entry (at 49.53 66.04) (size 2.54 2.54)
+  (bus_entry (at 49.53 71.12) (size 2.54 -2.54)
     (stroke (width 0) (type default))
   )
@@
     (stroke (width 0) (type default))
   )
-  (bus (pts (xy 49.53 66.04) (xy 49.53 74.93))
-    (stroke (width 0) (type default))
-  )
+  (bus (pts (xy 49.53 71.12) (xy 49.53 74.93))
+    (stroke (width 0) (type default))
+  )
