File: KiCad/NR24_Schematic/AMS.kicad_sch (KiCad schematic)
At the start: 4 parts

Commit message: v4
Connections:
- net TI Board: now reaches U?.2 (Ready_Power)
- net TI Board: now also U?.2 (Ready_Power), U?.4 (Charge_Power), U?.4 (Charge_Power)
- net Charge Sig: now reaches U?.5 (Charger_Safety)
- net Charge Sig: now also U?.5 (Charger_Safety)
- net AIR Input renamed AIR
- net Battery High out renamed HV +
- net Battery Low In renamed HV -
- net CAN_Ground renamed CAN_GND
- removed net Charging Port: U?.4 (Charge_Power), U?.5 (Charger_Safety)
- removed net Ti Board: U?.1 (Charge_Enable), U?.2 (Ready_Power), U?.3 (Discharge_Enable), U?.4 (Charge_Power)
Changed lines of the file:
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@@
+    (stroke (width 0) (type default))
+  )
+  (wire (pts (xy 166.37 92.71) (xy 166.37 113.03))
     (stroke (width 0) (type default))
   )
@@
   )
   (wire (pts (xy 181.61 85.09) (xy 161.29 85.09))
-    (stroke (width 0) (type default))
-  )
-  (wire (pts (xy 166.37 92.71) (xy 166.37 113.03))
     (stroke (width 0) (type default))
   )
@@
     (effects (font (size 4 4) (thickness 0.8) bold (color 0 0 0 1)))
   )
-  (global_label "Charging Port" (shape input) (at 143.51 113.03 270) (fields_autoplaced)
-    (effects (font (size 1.27 1.27)) (justify right))
-    (property "Intersheetrefs" "${INTERSHEET_REFS}" (at 143.51 129.3197 90)
-      (effects (font (size 1.27 1.27)) (justify right) hide)
-    )
-  )
-  (global_label "CAN_High" (shape input) (at 167.64 46.99 90) (fields_autoplaced)
-    (effects (font (size 1.27 1.27)) (justify left))
-    (property "Intersheetrefs" "${INTERSHEET_REFS}" (at 167.64 35.1148 90)
-      (effects (font (size 1.27 1.27)) (justify left) hide)
-    )
-  )
-  (global_label "Battery Low In" (shape input) (at 110.49 151.13 180) (fields_autoplaced)
-    (effects (font (size 1.27 1.27)) (justify right))
-    (property "Intersheetrefs" "${INTERSHEET_REFS}" (at 93.5954 151.13 0)
-      (effects (font (size 1.27 1.27)) (justify right) hide)
-    )
-  )
-  (global_label "CAN_Ground" (shape input) (at 172.72 46.99 90) (fields_autoplaced)
-    (effects (font (size 1.27 1.27)) (justify left))
-    (property "Intersheetrefs" "${INTERSHEET_REFS}" (at 172.72 32.6959 90)
-      (effects (font (size 1.27 1.27)) (justify left) hide)
-    )
-  )
-  (global_label "Ti Board" (shape input) (at 146.05 113.03 270) (fields_autoplaced)
-    (effects (font (size 1.27 1.27)) (justify right))
-    (property "Intersheetrefs" "${INTERSHEET_REFS}" (at 146.05 124.0584 90)
-      (effects (font (size 1.27 1.27)) (justify right) hide)
-    )
-  )
-  (global_label "Charging Port" (shape input) (at 166.37 113.03 270) (fields_autoplaced)
-    (effects (font (size 1.27 1.27)) (justify right))
-    (property "Intersheetrefs" "${INTERSHEET_REFS}" (at 166.37 129.3197 90)
-      (effects (font (size 1.27 1.27)) (justify left) hide)
-    )
-  )
-  (global_label "Ti Board" (shape input) (at 163.83 113.03 270) (fields_autoplaced)
-    (effects (font (size 1.27 1.27)) (justify right))
-    (property "Intersheetrefs" "${INTERSHEET_REFS}" (at 163.83 124.0584 90)
-      (effects (font (size 1.27 1.27)) (justify left) hide)
-    )
-  )
-  (global_label "CAN_Low" (shape input) (at 170.18 46.99 90) (fields_autoplaced)
-    (effects (font (size 1.27 1.27)) (justify left))
-    (property "Intersheetrefs" "${INTERSHEET_REFS}" (at 170.18 35.8405 90)
-      (effects (font (size 1.27 1.27)) (justify left) hide)
-    )
-  )
-  (global_label "AIR Input" (shape input) (at 182.88 29.21 270) (fields_autoplaced)
-    (effects (font (size 1.27 1.27)) (justify right))
-    (property "Intersheetrefs" "${INTERSHEET_REFS}" (at 182.88 40.9037 90)
-      (effects (font (size 1.27 1.27)) (justify right) hide)
-    )
-  )
-  (global_label "Battery High out" (shape input) (at 205.74 139.7 0) (fields_autoplaced)
-    (effects (font (size 1.27 1.27)) (justify left))
-    (property "Intersheetrefs" "${INTERSHEET_REFS}" (at 224.6302 139.7 0)
-      (effects (font (size 1.27 1.27)) (justify left) hide)
-    )
-  )
-  (global_label "Ti Board" (shape input) (at 158.75 113.03 270) (fields_autoplaced)
-    (effects (font (size 1.27 1.27)) (justify right))
-    (property "Intersheetrefs" "${INTERSHEET_REFS}" (at 158.75 124.0584 90)
-      (effects (font (size 1.27 1.27)) (justify left) hide)
-    )
-  )
-  (global_label "Ti Board" (shape input) (at 151.13 113.03 270) (fields_autoplaced)
-    (effects (font (size 1.27 1.27)) (justify right))
-    (property "Intersheetrefs" "${INTERSHEET_REFS}" (at 151.13 124.0584 90)
-      (effects (font (size 1.27 1.27)) (justify right) hide)
-    )
+  (hierarchical_label "TI Board" (shape input) (at 146.05 113.03 270) (fields_autoplaced)
+    (effects (font (size 1.27 1.27)) (justify right))
+  )
+  (hierarchical_label "HV -" (shape input) (at 110.49 151.13 180) (fields_autoplaced)
+    (effects (font (size 1.27 1.27)) (justify right))
+  )
+  (hierarchical_label "TI Board" (shape input) (at 166.37 113.03 270) (fields_autoplaced)
+    (effects (font (size 1.27 1.27)) (justify right))
+  )
+  (hierarchical_label "Charge Sig" (shape input) (at 168.91 113.03 270) (fields_autoplaced)
+    (effects (font (size 1.27 1.27)) (justify right))
+  )
+  (hierarchical_label "Charge Sig" (shape input) (at 143.51 113.03 270) (fields_autoplaced)
+    (effects (font (size 1.27 1.27)) (justify right))
+  )
+  (hierarchical_label "CAN_High" (shape input) (at 167.64 46.99 90) (fields_autoplaced)
+    (effects (font (size 1.27 1.27)) (justify left))
+  )
+  (hierarchical_label "TI Board" (shape input) (at 161.29 113.03 270) (fields_autoplaced)
+    (effects (font (size 1.27 1.27)) (justify right))
+  )
+  (hierarchical_label "HV +" (shape input) (at 205.74 139.7 0) (fields_autoplaced)
+    (effects (font (size 1.27 1.27)) (justify left))
+  )
+  (hierarchical_label "TI Board" (shape input) (at 151.13 113.03 270) (fields_autoplaced)
+    (effects (font (size 1.27 1.27)) (justify right))
+  )
+  (hierarchical_label "CAN_GND" (shape input) (at 172.72 46.99 90) (fields_autoplaced)
+    (effects (font (size 1.27 1.27)) (justify left))
+  )
+  (hierarchical_label "AIR" (shape input) (at 182.88 29.21 270) (fields_autoplaced)
+    (effects (font (size 1.27 1.27)) (justify right))
+  )
+  (hierarchical_label "CAN_Low" (shape input) (at 170.18 46.99 90) (fields_autoplaced)
+    (effects (font (size 1.27 1.27)) (justify left))
   )
   (symbol (lib_id "Device:Battery") (at 193.04 144.78 0) (mirror y) (unit 1)
