File: KiCad/NR24_Schematic/IMD.kicad_sch (KiCad schematic)
At the start: 4 parts

Commit message: v4
Connections:
- net Line output row is gone; now on net LV_High: U?.2 (Supply_Voltage)
- net 12V Low Voltage renamed LV_High
- net AIR Loop In renamed AIR_In
- net AIR Loop Out renamed AIR_Out
- net Dash Error Light renamed Dash_Error +
- net Dash_Error +: no longer U?.1 (STDP1)
- net Ground renamed GND
- net Line output high renamed HV_High
- new net Dash_Error -: U?.1 (STDP1)
- new net HV_Low: U?.2 (Supply_Voltage)
Changed lines of the file:
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@@
     (effects (font (size 4 4) (thickness 0.8) bold (color 0 0 0 1)))
   )
-  (global_label "Dash Error Light" (shape input) (at 162.56 59.69 180) (fields_autoplaced)
+  (hierarchical_label "LV_High" (shape input) (at 110.49 44.45 90) (fields_autoplaced)
+    (effects (font (size 1.27 1.27)) (justify left))
+  )
+  (hierarchical_label "AIR_In" (shape input) (at 162.56 77.47 180) (fields_autoplaced)
     (effects (font (size 1.27 1.27)) (justify right))
-    (property "Intersheetrefs" "${INTERSHEET_REFS}" (at 143.7303 59.69 0)
-      (effects (font (size 1.27 1.27)) (justify right) hide)
-    )
   )
-  (global_label "Line output row" (shape input) (at 45.72 90.17 90) (fields_autoplaced)
+  (hierarchical_label "GND" (shape input) (at 107.95 44.45 90) (fields_autoplaced)
     (effects (font (size 1.27 1.27)) (justify left))
-    (property "Intersheetrefs" "${INTERSHEET_REFS}" (at 45.72 72.066 90)
-      (effects (font (size 1.27 1.27)) (justify left) hide)
-    )
   )
-  (global_label "Ground" (shape input) (at 107.95 44.45 90) (fields_autoplaced)
+  (hierarchical_label "Dash_Error +" (shape input) (at 162.56 59.69 180) (fields_autoplaced)
+    (effects (font (size 1.27 1.27)) (justify right))
+  )
+  (hierarchical_label "HV_Low" (shape input) (at 45.72 90.17 90) (fields_autoplaced)
+    (effects (font (size 2 2)) (justify left))
+  )
+  (hierarchical_label "GND" (shape input) (at 195.58 90.17 0) (fields_autoplaced)
     (effects (font (size 1.27 1.27)) (justify left))
-    (property "Intersheetrefs" "${INTERSHEET_REFS}" (at 107.95 34.8126 90)
-      (effects (font (size 1.27 1.27)) (justify left) hide)
-    )
   )
-  (global_label "Ground" (shape input) (at 113.03 44.45 90) (fields_autoplaced)
+  (hierarchical_label "AIR_Out" (shape input) (at 162.56 81.28 180) (fields_autoplaced)
+    (effects (font (size 1.27 1.27)) (justify right))
+  )
+  (hierarchical_label "GND" (shape input) (at 115.57 44.45 90) (fields_autoplaced)
     (effects (font (size 1.27 1.27)) (justify left))
-    (property "Intersheetrefs" "${INTERSHEET_REFS}" (at 113.03 34.8126 90)
-      (effects (font (size 1.27 1.27)) (justify left) hide)
-    )
   )
-  (global_label "Dash Error Light" (shape input) (at 162.56 63.5 180) (fields_autoplaced)
+  (hierarchical_label "Dash_Error -" (shape input) (at 162.56 63.5 180) (fields_autoplaced)
     (effects (font (size 1.27 1.27)) (justify right))
-    (property "Intersheetrefs" "${INTERSHEET_REFS}" (at 143.7303 63.5 0)
-      (effects (font (size 1.27 1.27)) (justify right) hide)
-    )
   )
-  (global_label "Ground" (shape input) (at 115.57 44.45 90) (fields_autoplaced)
+  (hierarchical_label "HV_High" (shape input) (at 52.07 90.17 90) (fields_autoplaced)
+    (effects (font (size 2 2)) (justify left))
+  )
+  (hierarchical_label "GND" (shape input) (at 113.03 44.45 90) (fields_autoplaced)
     (effects (font (size 1.27 1.27)) (justify left))
-    (property "Intersheetrefs" "${INTERSHEET_REFS}" (at 115.57 34.8126 90)
-      (effects (font (size 1.27 1.27)) (justify left) hide)
-    )
-  )
-  (global_label "Line output high" (shape input) (at 52.07 90.17 90) (fields_autoplaced)
-    (effects (font (size 1.27 1.27)) (justify left))
-    (property "Intersheetrefs" "${INTERSHEET_REFS}" (at 52.07 71.2799 90)
-      (effects (font (size 1.27 1.27)) (justify left) hide)
-    )
-  )
-  (global_label "12V Low Voltage" (shape input) (at 110.49 44.45 90) (fields_autoplaced)
-    (effects (font (size 1.27 1.27)) (justify left))
-    (property "Intersheetrefs" "${INTERSHEET_REFS}" (at 110.49 25.4993 90)
-      (effects (font (size 1.27 1.27)) (justify left) hide)
-    )
-  )
-  (global_label "Ground" (shape input) (at 195.58 90.17 0) (fields_autoplaced)
-    (effects (font (size 1.27 1.27)) (justify left))
-    (property "Intersheetrefs" "${INTERSHEET_REFS}" (at 205.2174 90.17 0)
-      (effects (font (size 1.27 1.27)) (justify left) hide)
-    )
-  )
-  (global_label "AIR Loop Out" (shape input) (at 162.56 81.28 180) (fields_autoplaced)
-    (effects (font (size 1.27 1.27)) (justify right))
-    (property "Intersheetrefs" "${INTERSHEET_REFS}" (at 146.9959 81.28 0)
-      (effects (font (size 1.27 1.27)) (justify right) hide)
-    )
-  )
-  (global_label "AIR Loop In" (shape input) (at 162.56 77.47 180) (fields_autoplaced)
-    (effects (font (size 1.27 1.27)) (justify right))
-    (property "Intersheetrefs" "${INTERSHEET_REFS}" (at 148.4473 77.47 0)
-      (effects (font (size 1.27 1.27)) (justify right) hide)
-    )
   )
   (symbol (lib_id "Diode:1N4001") (at 194.31 81.28 270) (unit 1)
