File: KiCad/NR24_Schematic/Ti_Board.kicad_sch (KiCad schematic)
At the start: 2 parts, among them J5 Dash TI Connection, J8 CAN Connector

Commit message: B-? where are stops connected to
Changed lines of the file:
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@@
   (no_connect (at 186.69 82.55))
   (no_connect (at 116.84 82.55))
+  (wire (pts (xy 90.17 74.93) (xy 104.14 74.93))
+    (stroke (width 0) (type default))
+  )
+  (bus (pts (xy 99.06 82.55) (xy 99.06 45.72))
+    (stroke (width 0) (type default))
+  )
   (wire (pts (xy 91.44 85.09) (xy 104.14 85.09))
+    (stroke (width 0) (type default))
+  )
+  (wire (pts (xy 91.44 80.01) (xy 104.14 80.01))
+    (stroke (width 0) (type default))
+  )
+  (wire (pts (xy 91.44 77.47) (xy 104.14 77.47))
+    (stroke (width 0) (type default))
+  )
+  (bus (pts (xy 95.25 45.72) (xy 99.06 45.72))
+    (stroke (width 0) (type default))
+  )
+  (wire (pts (xy 90.17 72.39) (xy 104.14 72.39))
+    (stroke (width 0) (type default))
+  )
+  (wire (pts (xy 92.71 82.55) (xy 104.14 82.55))
     (stroke (width 0) (type default))
   )
@@
     (stroke (width 0) (type default))
   )
-  (global_label "F_Light(-)" (shape input) (at 104.14 77.47 180) (fields_autoplaced)
+  (global_label "F_Light(-)" (shape input) (at 91.44 77.47 180) (fields_autoplaced)
     (effects (font (size 1.27 1.27) (thickness 0.254) bold) (justify right))
-    (property "Intersheetrefs" "${INTERSHEET_REFS}" (at 90.7002 77.47 0)
+    (property "Intersheetrefs" "${INTERSHEET_REFS}" (at 78.0002 77.47 0)
       (effects (font (size 1.27 1.27) (thickness 0.254) bold) (justify right) hide)
     )
   )
-  (global_label "F_Light(+)" (shape input) (at 104.14 74.93 180) (fields_autoplaced)
+  (global_label "F_Light(+)" (shape input) (at 90.17 74.93 180) (fields_autoplaced)
     (effects (font (size 1.27 1.27) (thickness 0.254) bold) (justify right))
-    (property "Intersheetrefs" "${INTERSHEET_REFS}" (at 90.7002 74.93 0)
+    (property "Intersheetrefs" "${INTERSHEET_REFS}" (at 76.7302 74.93 0)
       (effects (font (size 1.27 1.27) (thickness 0.254) bold) (justify right) hide)
     )
@@
     )
   )
-  (global_label "N_Light(-)" (shape input) (at 104.14 82.55 180) (fields_autoplaced)
+  (global_label "N_Light(-)" (shape input) (at 92.71 82.55 180) (fields_autoplaced)
     (effects (font (size 1.27 1.27) (thickness 0.254) bold) (justify right))
-    (property "Intersheetrefs" "${INTERSHEET_REFS}" (at 90.4583 82.55 0)
+    (property "Intersheetrefs" "${INTERSHEET_REFS}" (at 79.0283 82.55 0)
       (effects (font (size 1.27 1.27) (thickness 0.254) bold) (justify right) hide)
     )
@@
     )
   )
-  (global_label "Rocker_3" (shape input) (at 104.14 72.39 180) (fields_autoplaced)
+  (global_label "Rocker_3" (shape input) (at 90.17 72.39 180) (fields_autoplaced)
     (effects (font (size 1.27 1.27) (thickness 0.254) bold) (justify right))
-    (property "Intersheetrefs" "${INTERSHEET_REFS}" (at 92.0912 72.39 0)
+    (property "Intersheetrefs" "${INTERSHEET_REFS}" (at 78.1212 72.39 0)
       (effects (font (size 1.27 1.27) (thickness 0.254) bold) (justify right) hide)
     )
@@
     )
   )
-  (global_label "N_Light(+)" (shape input) (at 104.14 80.01 180) (fields_autoplaced)
+  (global_label "N_Light(+)" (shape input) (at 91.44 80.01 180) (fields_autoplaced)
     (effects (font (size 1.27 1.27) (thickness 0.254) bold) (justify right))
-    (property "Intersheetrefs" "${INTERSHEET_REFS}" (at 90.4583 80.01 0)
+    (property "Intersheetrefs" "${INTERSHEET_REFS}" (at 77.7583 80.01 0)
       (effects (font (size 1.27 1.27) (thickness 0.254) bold) (justify right) hide)
     )

Commit message: Please finish connection and AIR coils
Parts:
- added J6: SpeakON_NL2, symbol Connector_Audio:SpeakON_NL2
Connections:
- new net GND: J6.1-
- new net Ready to Drive Speaker (+): J6.1+
Changed lines of the file:
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@@
   (no_connect (at 186.69 82.55))
   (no_connect (at 116.84 82.55))
+  (wire (pts (xy 129.54 36.83) (xy 129.54 33.02))
+    (stroke (width 0) (type default))
+  )
   (wire (pts (xy 90.17 74.93) (xy 104.14 74.93))
     (stroke (width 0) (type default))
   )
+  (wire (pts (xy 113.03 44.45) (xy 121.92 44.45))
+    (stroke (width 0) (type default))
+  )
   (bus (pts (xy 99.06 82.55) (xy 99.06 45.72))
     (stroke (width 0) (type default))
@@
     (stroke (width 0) (type default))
   )
+  (wire (pts (xy 114.3 33.02) (xy 129.54 33.02))
+    (stroke (width 0) (type default))
+  )
   (wire (pts (xy 91.44 99.06) (xy 91.44 85.09))
     (stroke (width 0) (type default))
@@
     (property "Intersheetrefs" "${INTERSHEET_REFS}" (at 76.7302 74.93 0)
       (effects (font (size 1.27 1.27) (thickness 0.254) bold) (justify right) hide)
+    )
+  )
+  (global_label "GND" (shape input) (at 118.11 44.45 90) (fields_autoplaced)
+    (effects (font (size 1.27 1.27)) (justify left))
+    (property "Intersheetrefs" "${INTERSHEET_REFS}" (at 118.11 37.5943 90)
+      (effects (font (size 1.27 1.27)) (justify left) hide)
     )
   )
@@
     (property "Intersheetrefs" "${INTERSHEET_REFS}" (at 79.0283 82.55 0)
       (effects (font (size 1.27 1.27) (thickness 0.254) bold) (justify right) hide)
+    )
+  )
+  (global_label "Ready to Drive Speaker (+)" (shape input) (at 129.54 33.02 0) (fields_autoplaced)
+    (effects (font (size 1.27 1.27)) (justify left))
+    (property "Intersheetrefs" "${INTERSHEET_REFS}" (at 159.3765 33.02 0)
+      (effects (font (size 1.27 1.27)) (justify left) hide)
     )
   )
@@
         )
       )
+    )
+  )
+  (symbol (lib_id "Connector_Audio:SpeakON_NL2") (at 129.54 44.45 0) (unit 1)
+    (in_bom yes) (on_board yes) (dnp no) (fields_autoplaced)
+    (property "Reference" "J6" (at 135.89 43.18 0)
+      (effects (font (size 1.27 1.27)) (justify left))
+    )
+    (property "Value" "SpeakON_NL2" (at 135.89 45.72 0)
+      (effects (font (size 1.27 1.27)) (justify left))
+    )
+    (property "Footprint" "" (at 129.54 44.45 0)
+      (effects (font (size 1.27 1.27)) hide)
+    )
+    (property "Datasheet" "http://www.neutrik.com/en/speakon/" (at 129.54 44.45 0)
+      (effects (font (size 1.27 1.27)) hide)
+    )
+    (pin "1-")
+    (pin "1+")
+    (instances
+      (project "Car_TractiveSystem_v2"
+        (path "/588b5c14-1813-4e1d-9dbe-940839ecebe3/42103732-fa28-467e-b394-54af70cbf903"
+          (reference "J6") (unit 1)
+        )
+      )

Commit message: Please Finish Dash
Connections:
- net CAN_GND_fromBattery: no longer J8.9 (Pin_9)
- net CAN_High_fromBattery: no longer J8.3 (Pin_3)
- net CAN_High_fromSevcon: no longer J8.2 (Pin_2)
- net CAN_High_toDisplay: no longer J8.1 (Pin_1)
- net CAN_Low_fromBattery: no longer J8.10 (Pin_10)
- net CAN_Low_fromSevcon: no longer J8.11 (Pin_11)
- net CAN_Low_toDisplay: no longer J8.12 (Pin_12)
- net CAN_PWR_fromBattery: no longer J8.4 (Pin_4)
- net CAN_PWR_fromSevcon: no longer J8.5 (Pin_5)
- net F_Light(+): no longer J5.2 (Pin_2)
- net F_Light(-): no longer J5.3 (Pin_3)
- net N_Light(+): no longer J5.4 (Pin_4)
- net N_Light(-): no longer J5.5 (Pin_5)
- net Rocker_3: no longer J5.1 (Pin_1)
- net system_on_fromBattery: no longer J8.7 (Pin_7)
- net throttle_en_fromBattery: no longer J8.6 (Pin_6)
Other:
- note added: "11 wires"
- note added: "throttle_en and system_on connected to 5V off of the TI board (~20mA)"
- moved on the sheet: J8

Commit message: t
Parts:
- added J5: J8 Pin J6 Pin, symbol Connector_Generic:Conn_02x06_Counter_Clockwise
- added J5: J1 Pin J3 Pin, symbol Connector_Generic:Conn_02x06_Counter_Clockwise
- added J5: J5 Pin J7 Pin, symbol Connector_Generic:Conn_02x06_Counter_Clockwise
- added J5: J4 Pin J2 Pin, symbol Connector_Generic:Conn_02x06_Counter_Clockwise
Changed lines of the file:
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@@
+    )
+  )
+  (symbol (lib_name "Conn_02x06_Counter_Clockwise_4") (lib_id "Connector_Generic:Conn_02x06_Counter_Clockwise") (at 210.82 123.19 0) (unit 1)
+    (in_bom yes) (on_board yes) (dnp no)
+    (property "Reference" "J5" (at 207.01 134.62 90)
+      (effects (font (size 1.27 1.27)) (justify right) hide)
+    )
+    (property "Value" "J8 Pin	J6 Pin" (at 204.47 146.05 0)
+      (effects (font (size 1.27 1.27)) (justify left))
+    )
+    (property "Footprint" "" (at 210.82 123.19 0)
+      (effects (font (size 1.27 1.27)) hide)
+    )
+    (property "Datasheet" "~" (at 210.82 123.19 0)
+      (effects (font (size 1.27 1.27)) hide)
+    )
+    (pin "51")
+    (pin "52")
+    (pin "53")
+    (pin "54")
+    (pin "55")
+    (pin "56")
+    (pin "57")
+    (pin "58")
+    (pin "59")
+    (pin "60")
+    (pin "71")
+    (pin "72")
+    (pin "73")
+    (pin "74")
+    (pin "75")
+    (pin "76")
+    (pin "77")
+    (pin "78")
+    (pin "79")
+    (pin "80")
+    (instances
+      (project "Car_TractiveSystem_v2"
+        (path "/588b5c14-1813-4e1d-9dbe-940839ecebe3"
+          (reference "J5") (unit 1)
+        )
+        (path "/588b5c14-1813-4e1d-9dbe-940839ecebe3/42103732-fa28-467e-b394-54af70cbf903"
+          (reference "J13") (unit 1)
+        )
+      )
+      (project "Ti_Board"
+        (path "/95cd4c17-85c0-46ed-9908-1b2dc6d240f0"
+          (reference "J4") (unit 1)
+        )
+      )
+    )
+  )
+  (symbol (lib_name "Conn_02x06_Counter_Clockwise_1") (lib_id "Connector_Generic:Conn_02x06_Counter_Clockwise") (at 118.11 123.19 0) (unit 1)
+    (in_bom yes) (on_board yes) (dnp no)
+    (property "Reference" "J5" (at 114.3 134.62 90)
+      (effects (font (size 1.27 1.27)) (justify right) hide)
+    )
+    (property "Value" "J1 Pin	J3 Pin" (at 111.76 146.05 0)
+      (effects (font (size 1.27 1.27)) (justify left))
+    )
+    (property "Footprint" "" (at 118.11 123.19 0)
+      (effects (font (size 1.27 1.27)) hide)
+    )
+    (property "Datasheet" "~" (at 118.11 123.19 0)
+      (effects (font (size 1.27 1.27)) hide)
+    )
+    (pin "1")
+    (pin "10")
+    (pin "2")
+    (pin "21")
+    (pin "22")
+    (pin "23")
+    (pin "24")
+    (pin "25")
+    (pin "26")
+    (pin "27")
+    (pin "28")
+    (pin "29")
+    (pin "3")
+    (pin "30")
+    (pin "4")
+    (pin "5")
+    (pin "6")
+    (pin "7")
+    (pin "8")
+    (pin "9")
+    (instances
+      (project "Car_TractiveSystem_v2"
+        (path "/588b5c14-1813-4e1d-9dbe-940839ecebe3"
+          (reference "J5") (unit 1)
+        )
+        (path "/588b5c14-1813-4e1d-9dbe-940839ecebe3/42103732-fa28-467e-b394-54af70cbf903"
+          (reference "J10") (unit 1)
+        )
+      )
+      (project "Ti_Board"
+        (path "/95cd4c17-85c0-46ed-9908-1b2dc6d240f0"
+          (reference "J1") (unit 1)
+        )
+      )
     )
   )
@@
         )
       )
+      (project "Ti_Board"
+        (path "/95cd4c17-85c0-46ed-9908-1b2dc6d240f0"
+          (reference "J8") (unit 1)
+        )
+      )
+    )
+  )
+  (symbol (lib_name "Conn_02x06_Counter_Clockwise_3") (lib_id "Connector_Generic:Conn_02x06_Counter_Clockwise") (at 180.34 123.19 0) (unit 1)
+    (in_bom yes) (on_board yes) (dnp no)
+    (property "Reference" "J5" (at 176.53 134.62 90)
+      (effects (font (size 1.27 1.27)) (justify right) hide)
+    )
+    (property "Value" "J5 Pin	J7 Pin" (at 173.99 146.05 0)
+      (effects (font (size 1.27 1.27)) (justify left))
+    )
+    (property "Footprint" "" (at 180.34 123.19 0)
+      (effects (font (size 1.27 1.27)) hide)
+    )
+    (property "Datasheet" "~" (at 180.34 123.19 0)
+      (effects (font (size 1.27 1.27)) hide)
+    )
+    (pin "41")
+    (pin "42")
+    (pin "43")
+    (pin "44")
+    (pin "45")
+    (pin "46")
+    (pin "47")
+    (pin "48")
+    (pin "49")
+    (pin "50")
+    (pin "61")
+    (pin "62")
+    (pin "63")
+    (pin "64")
+    (pin "65")
+    (pin "66")
+    (pin "67")
+    (pin "68")
+    (pin "69")
+    (pin "70")
+    (instances
+      (project "Car_TractiveSystem_v2"
+        (path "/588b5c14-1813-4e1d-9dbe-940839ecebe3"
+          (reference "J5") (unit 1)
+        )
+        (path "/588b5c14-1813-4e1d-9dbe-940839ecebe3/42103732-fa28-467e-b394-54af70cbf903"
+          (reference "J12") (unit 1)
+        )
+      )
+      (project "Ti_Board"
+        (path "/95cd4c17-85c0-46ed-9908-1b2dc6d240f0"
+          (reference "J3") (unit 1)
+        )
+      )
     )
   )
@@
         (path "/588b5c14-1813-4e1d-9dbe-940839ecebe3/42103732-fa28-467e-b394-54af70cbf903"
           (reference "J6") (unit 1)
+        )
+      )
+      (project "Ti_Board"
+        (path "/95cd4c17-85c0-46ed-9908-1b2dc6d240f0"
+          (reference "J6") (unit 1)
+        )
+      )
+    )
+  )
+  (symbol (lib_name "Conn_02x06_Counter_Clockwise_2") (lib_id "Connector_Generic:Conn_02x06_Counter_Clockwise") (at 149.86 123.19 0) (unit 1)
+    (in_bom yes) (on_board yes) (dnp no)
+    (property "Reference" "J5" (at 146.05 134.62 90)
+      (effects (font (size 1.27 1.27)) (justify right) hide)
+    )
+    (property "Value" "J4 Pin	J2 Pin" (at 143.51 146.05 0)
+      (effects (font (size 1.27 1.27)) (justify left))
+    )
+    (property "Footprint" "" (at 149.86 123.19 0)
+      (effects (font (size 1.27 1.27)) hide)
+    )
+    (property "Datasheet" "~" (at 149.86 123.19 0)
+      (effects (font (size 1.27 1.27)) hide)
+    )
+    (pin "11")
+    (pin "12")
+    (pin "13")
+    (pin "14")
+    (pin "15")
+    (pin "16")
+    (pin "17")
+    (pin "18")
+    (pin "19")
+    (pin "20")
+    (pin "31")
+    (pin "32")
+    (pin "33")
+    (pin "34")
+    (pin "35")
+    (pin "36")
+    (pin "37")
+    (pin "38")
+    (pin "39")
+    (pin "40")
+    (instances
+      (project "Car_TractiveSystem_v2"
+        (path "/588b5c14-1813-4e1d-9dbe-940839ecebe3"
+          (reference "J5") (unit 1)
+        )
+        (path "/588b5c14-1813-4e1d-9dbe-940839ecebe3/42103732-fa28-467e-b394-54af70cbf903"
+          (reference "J11") (unit 1)
+        )
+      )
+      (project "Ti_Board"
+        (path "/95cd4c17-85c0-46ed-9908-1b2dc6d240f0"
+          (reference "J2") (unit 1)
         )
       )
@@
         )
       )
-    )
+      (project "Ti_Board"
+        (path "/95cd4c17-85c0-46ed-9908-1b2dc6d240f0"
+          (reference "J5") (unit 1)
+        )
+      )
+    )
+  )
+  (sheet_instances
+    (path "/" (page "1"))
   )
 )
